Commit message: addded new enviorment and lidar sensor

File: urdf/macros.xacro (robot description, xacro)
@@ -595,7 +595,77 @@
       </sensor>
     </gazebo>
+    <!-- ============== YDLIDAR X2 LiDAR ============== -->
+    <!-- Physical link representing the lidar unit on top of the rover -->
+    <link name="${link_prefix}lidar_link">
+      <inertial>
+        <mass value="0.150"/>
+        <origin xyz="0 0 0.048" rpy="0 0 0"/>
+        <inertia ixx="0.0001" ixy="0" ixz="0" iyy="0.0001" iyz="0" izz="0.00005"/>
+      </inertial>
+      <visual>
+        <origin xyz="0 0 0.048" rpy="0 0 0"/>
+        <geometry>
+          <cylinder radius="0.030" length="0.096"/>
+        </geometry>
+        <material name="lidar_black">
+          <color rgba="0.1 0.1 0.1 1.0"/>
+        </material>
+      </visual>
+      <collision>
+        <origin xyz="0 0 0.048" rpy="0 0 0"/>
+        <geometry>
+          <cylinder radius="0.030" length="0.096"/>
+        </geometry>
+      </collision>
+    </link>
+    <!-- Mount lidar on top of base_link -->
+    <joint name="${link_prefix}lidar_joint" type="fixed">
+      <origin xyz="0 0 0.06" rpy="0 0 0"/>
+      <parent link="${link_prefix}base_link"/>
+      <child link="${link_prefix}lidar_link"/>
+    </joint>
+    <!-- Gazebo gpu_lidar sensor matching YDLIDAR X2 specs -->
+    <gazebo reference="${link_prefix}lidar_link">
+      <sensor name="ydlidar_x2" type="gpu_lidar">
+        <always_on>1</always_on>
+        <update_rate>7</update_rate>
+        <visualize>true</visualize>
+        <topic>${link_prefix}scan</topic>
+        <gz_frame_id>${link_prefix}lidar_link</gz_frame_id>
+        <ray>
+          <scan>
+            <horizontal>
+              <samples>430</samples>
+              <resolution>1</resolution>
+              <min_angle>-3.14159</min_angle>
+              <max_angle>3.14159</max_angle>
+            </horizontal>
+            <vertical>
+              <samples>1</samples>
+              <resolution>1</resolution>
+              <min_angle>0</min_angle>
+              <max_angle>0</max_angle>
+            </vertical>
+          </scan>
+          <range>
+            <min>0.12</min>
+            <max>8.0</max>
+            <resolution>0.01</resolution>
+          </range>
+          <noise>
+            <type>gaussian</type>
+            <mean>0.0</mean>
+            <stddev>0.01</stddev>
+          </noise>
+        </ray>
+      </sensor>
+    </gazebo>
     <gazebo>
       <plugin filename="libgz-sim-imu-system.so"
               name="gz::sim::systems::Imu">
+      </plugin>
+      <plugin filename="libgz-sim-sensors-system.so"
+              name="gz::sim::systems::Sensors">
+        <render_engine>ogre2</render_engine>
       </plugin>
       <plugin
